Commit message: update simple_humanoid.urdf
with this fix, all the simple_humanoid tests pass with the only exception
of bcalc: each frame position is good, but the orientation is not, some
axis are permuted.

This is expected since the frame definitions are not identical.

The rnea and crba tests work as expected since they operate in configuration
space work.

The various jacobian tests also work because the compute the world
velocites of the links, not the body velocity.

File: data/simple_humanoid.urdf (robot description, URDF)
Before this commit: robot simple_humanoid, 31 links, 30 joints
Joints:
- joint WAIST_P: origin xyz=0 0 0.176 rpy=0 0 0 -> xyz=0 0 0 rpy=0 0 0
